Commit message: 增加moveit_bridge.py脚本，通过接口完成规划

File: urdf/lifting_platform.urdf.xacro (robot description, xacro)
@@ -65,5 +65,5 @@
   </link>
   <joint name="updown" type="prismatic">
-    <origin xyz="0 0 1.6" rpy="0 0 0"/>
+    <origin xyz="0.2 0 1.6" rpy="0 0 0"/>
     <parent link="base_link"/>
     <child link="column_Link"/>

Commit message: 调整运行速度

File: urdf/lifting_platform.urdf.xacro (robot description, xacro)
@@ -69,5 +69,5 @@
     <child link="column_Link"/>
     <axis xyz="0 0 -1"/>
-    <limit lower="0" upper="1.0" effort="930" velocity="0.3"/>
+    <limit lower="0" upper="1.0" effort="930" velocity="0.02"/>
     <dynamics damping="2.5" friction="15"/>
   </joint>

Commit message: 适配四横电机“

File: urdf/lifting_platform.urdf.xacro (robot description, xacro)
@@ -69,5 +69,5 @@
     <child link="column_Link"/>
     <axis xyz="0 0 -1"/>
-    <limit lower="0" upper="1.0" effort="930" velocity="0.02"/>
+    <limit lower="0" upper="1.0" effort="930" velocity="2"/>
     <dynamics damping="2.5" friction="15"/>
   </joint>
